Commit message: using ikpy lib for fwd and inv kinematics

File: config/awesome_crane.urdf (robot description, URDF)
Before this commit: robot crane, 5 links, 4 joints
Joints:
- joint lift_joint: limit lower=0 upper=1.5 effort=100 velocity=0.5 -> lower=-0.5 upper=1.5 effort=100 velocity=0.5

Commit message: adding basic frontend setup to print joint angles

File: config/awesome_crane.urdf (robot description, URDF)
Before this commit: robot crane, 5 links, 4 joints
Joints:
- joint elbow_joint: limit lower=-1.57 upper=1.57 effort=100 velocity=1.0 -> lower=-3.14 upper=3.14 effort=100 velocity=1.0; origin xyz=0.5 0 0 rpy=0 0 0 -> xyz=1.0 0 0 rpy=0 0 0
- joint lift_joint: limit lower=-0.5 upper=1.5 effort=100 velocity=0.5 -> lower=-0.1 upper=3.0 effort=100 velocity=0.05
- joint wrist_joint: limit lower=-1.57 upper=1.57 effort=100 velocity=1.0 -> lower=-3.14 upper=3.14 effort=100 velocity=1.0; origin xyz=0.5 0 -1 rpy=0 0 0 -> xyz=1.0 0 -1 rpy=0 0 0
