Commit message: adding last link

File: config/public/awesome_crane1.urdf (robot description, URDF)
Before this commit: robot crane, 5 links, 4 joints
Joints:
- joint lift_joint: origin xyz=0 0 0.125 rpy=0 0 0 -> xyz=0 0 0.375 rpy=0 0 0
- joint swing_joint: origin xyz=0 0 0.25 rpy=0 0 0 -> xyz=0 0 0 rpy=0 0 0
